File: kicad/grower_light/grower_light.sch (KiCad schematic (older format))
At the start: 14 parts, among them J1 Conn_01x06, J2 Temp, J3 Light, U1 ATMEGA328PB-AU, Y1 9,216 MHz

Commit message: Add source and update schematic
Parts:
- removed U1: ATMEGA328PB-AU, Package_QFP:TQFP-32_7x7mm_P0.8mm, symbol MCU_Atmel_ATMEGA:ATMEGA328PB-AU
- added C7, C8, C9: 100n, Capacitor_SMD:C_0805_2012Metric, symbol Device:C
- added J4: AVR_UART, Connector_PinHeader_2.54mm:PinHeader_1x03_P2.54mm_Vertical, symbol Connector_Generic:Conn_01x03
- added J5: ESP_UART, Connector_PinHeader_2.54mm:PinHeader_1x03_P2.54mm_Vertical, symbol Connector_Generic:Conn_01x03
- added L1: 100u, Inductor_SMD:L_0805_2012Metric, symbol Device:L
- added R4: 100, Resistor_SMD:R_0805_2012Metric, symbol Device:R
- added R5, R6: 10k, Resistor_SMD:R_0805_2012Metric, symbol Device:R
- added U1: ATMEGA328-AU, Package_QFP:TQFP-32_7x7mm_P0.8mm, symbol MCU_Atmel_ATMEGA:ATMEGA328-AU
- added U2: ESP-12_07v2, lib:ESP-07v2, symbol esp-12_07v2_08v2-rescue-esp8266_dht22:ESP-12_07v2_08v2-RESCUE-esp8266_dht22
Connections:
- net labels added: RX, TX
- net labels removed: GNDPWR
- wire segments 61 -> 108
- no-connect marks 0 -> 24

Commit message: Add ds1307 clock
Parts:
- added BT1: 3V, symbol Device:Battery_Cell
- added R7, R8: 4k7, Resistor_SMD:R_0805_2012Metric, symbol Device:R
- added U3: DS1307Z+, Package_SOIC:SO-8_5.3x6.2mm_P1.27mm, symbol maxim:DS1307Z+
- added Y2: 32768, Crystal:Crystal_SMD_MicroCrystal_CC4V-T1A-2Pin_5.0x1.9mm, symbol Device:Crystal
Connections:
- net labels added: SCL, SDA
- wire segments 108 -> 127
- no-connect marks 24 -> 23
Changed lines of the file:
@@
 L Connector_Generic:Conn_01x06 J1
 U 1 1 5A678FDE
-P 9200 1800
-F 0 "J1" H 9280 1792 50  0000 L CNN
-F 1 "Conn_01x06" H 9280 1701 50  0000 L CNN
-F 2 "Connector_PinHeader_2.54mm:PinHeader_2x03_P2.54mm_Vertical" H 9200 1800 50  0001 C CNN
-F 3 "~" H 9200 1800 50  0001 C CNN
-	1    9200 1800
+P 7150 1300
+F 0 "J1" H 7230 1292 50  0000 L CNN
+F 1 "Conn_01x06" H 7230 1201 50  0000 L CNN
+F 2 "Connector_PinHeader_2.54mm:PinHeader_2x03_P2.54mm_Vertical" H 7150 1300 50  0001 C CNN
+F 3 "~" H 7150 1300 50  0001 C CNN
+	1    7150 1300
 	1    0    0    -1
 $EndComp
@@
 L power:VCC #PWR07
 U 1 1 5A679056
-P 8650 1500
-F 0 "#PWR07" H 8650 1350 50  0001 C CNN
-F 1 "VCC" H 8667 1673 50  0000 C CNN
-F 2 "" H 8650 1500 50  0001 C CNN
-F 3 "" H 8650 1500 50  0001 C CNN
-	1    8650 1500
-	1    0    0    -1
-$EndComp
-Wire Wire Line
-	8650 1500 8650 1700
-Wire Wire Line
-	8650 1700 9000 1700
+P 6600 1000
+F 0 "#PWR07" H 6600 850 50  0001 C CNN
+F 1 "VCC" H 6617 1173 50  0000 C CNN
+F 2 "" H 6600 1000 50  0001 C CNN
+F 3 "" H 6600 1000 50  0001 C CNN
+	1    6600 1000
+	1    0    0    -1
+$EndComp
+Wire Wire Line
+	6600 1000 6600 1200
+Wire Wire Line
+	6600 1200 6950 1200
 $Comp
 L power:GND #PWR08
 U 1 1 5A6790A2
-P 8650 2200
-F 0 "#PWR08" H 8650 1950 50  0001 C CNN
-F 1 "GND" H 8655 2027 50  0000 C CNN
-F 2 "" H 8650 2200 50  0001 C CNN
-F 3 "" H 8650 2200 50  0001 C CNN
-	1    8650 2200
-	1    0    0    -1
-$EndComp
-Wire Wire Line
-	8650 2200 8650 2100
-Wire Wire Line
-	8650 2100 9000 2100
-Wire Wire Line
-	9000 1600 8800 1600
-Wire Wire Line
-	9000 1800 8800 1800
-Wire Wire Line
-	9000 1900 8800 1900
-Wire Wire Line
-	9000 2000 8800 2000
+P 6600 1700
+F 0 "#PWR08" H 6600 1450 50  0001 C CNN
+F 1 "GND" H 6605 1527 50  0000 C CNN
+F 2 "" H 6600 1700 50  0001 C CNN
+F 3 "" H 6600 1700 50  0001 C CNN
+	1    6600 1700
+	1    0    0    -1
+$EndComp
+Wire Wire Line
+	6600 1700 6600 1600
+Wire Wire Line
+	6600 1600 6950 1600
+Wire Wire Line
+	6950 1100 6750 1100
+Wire Wire Line
+	6950 1300 6750 1300
+Wire Wire Line
+	6950 1400 6750 1400
+Wire Wire Line
+	6950 1500 6750 1500
 Wire Wire Line
 	5500 2400 5700 2400
@@
 Text Label 5400 1150 0    50   ~ 0
 RES
-Text Label 8800 1600 0    50   ~ 0
+Text Label 6750 1100 0    50   ~ 0
 MISO
-Text Label 8800 1800 0    50   ~ 0
+Text Label 6750 1300 0    50   ~ 0
 SCK
-Text Label 8800 1900 0    50   ~ 0
+Text Label 6750 1400 0    50   ~ 0
 MOSI
-Text Label 8800 2000 0    50   ~ 0
+Text Label 6750 1500 0    50   ~ 0
 RES
 $Comp
@@
 NoConn ~ 5500 2950
 NoConn ~ 5500 3050
-NoConn ~ 5500 3150
-NoConn ~ 5500 3250
 NoConn ~ 5500 3700
 NoConn ~ 5500 3800
@@
 NoConn ~ 10050 4150
 NoConn ~ 10050 4250
+$Comp
+L maxim:DS1307Z+ U3
+U 1 1 5A695BF6
+P 9450 1650
+F 0 "U3" H 9000 2200 50  0000 C CNN
+F 1 "DS1307Z+" H 9750 2200 50  0000 C CNN
+F 2 "Package_SOIC:SO-8_5.3x6.2mm_P1.27mm" H 9450 1650 50  0001 C CNN
+F 3 "" H 9450 1650 50  0001 C CNN
+	1    9450 1650
+	1    0    0    -1
+$EndComp
+$Comp
+L power:GND #PWR031
+U 1 1 5A698FC0
+P 9450 2450
+F 0 "#PWR031" H 9450 2200 50  0001 C CNN
+F 1 "GND" H 9455 2277 50  0000 C CNN
+F 2 "" H 9450 2450 50  0001 C CNN
+F 3 "" H 9450 2450 50  0001 C CNN
+	1    9450 2450
+	1    0    0    -1
+$EndComp
+Wire Wire Line
+	9450 2450 9450 2250
+$Comp
+L power:VCC #PWR030
+U 1 1 5A69C12F
+P 9450 850
+F 0 "#PWR030" H 9450 700 50  0001 C CNN
+F 1 "VCC" H 9467 1023 50  0000 C CNN
+F 2 "" H 9450 850 50  0001 C CNN
+F 3 "" H 9450 850 50  0001 C CNN
+	1    9450 850
+	1    0    0    -1
+$EndComp
+Wire Wire Line
+	9450 850  9450 1050
+Wire Wire Line
+	8250 1350 8450 1350
+Text Label 8250 1350 0    50   ~ 0
+SCL
+Text Label 8250 1550 0    50   ~ 0
+SDA
+$Comp
+L Device:Crystal Y2
+U 1 1 5A6A5E18
+P 8400 1850
+F 0 "Y2" H 8150 1900 50  0000 C CNN
+F 1 "32768" H 8650 1900 50  0000 C CNN
+F 2 "Crystal:Crystal_SMD_MicroCrystal_CC4V-T1A-2Pin_5.0x1.9mm" H 8400 1850 50  0001 C CNN
+F 3 "" H 8400 1850 50  0001 C CNN
+	1    8400 1850
+	1    0    0    -1
+$EndComp
+Wire Wire Line
+	8550 1850 8850 1850
+Wire Wire Line
+	8250 1850 8100 1850
+Wire Wire Line
+	8100 1850 8100 2050
+Wire Wire Line
+	8100 2050 8850 2050
+$Comp
+L Device:Battery_Cell BT1
+U 1 1 5A6ACC33
+P 10550 2250
+F 0 "BT1" H 10668 2346 50  0000 L CNN
+F 1 "3V" H 10668 2255 50  0000 L CNN
+F 2 "" V 10550 2310 50  0001 C CNN
+F 3 "" V 10550 2310 50  0001 C CNN
+	1    10550 2250
+	1    0    0    -1
+$EndComp
+Wire Wire Line
+	10550 2050 10550 1950
+Wire Wire Line
+	10550 1950 10050 1950
+$Comp
+L power:GND #PWR032
+U 1 1 5A6B055A
+P 10550 2450
+F 0 "#PWR032" H 10550 2200 50  0001 C CNN
+F 1 "GND" H 10555 2277 50  0000 C CNN
+F 2 "" H 10550 2450 50  0001 C CNN
+F 3 "" H 10550 2450 50  0001 C CNN
+	1    10550 2450
+	1    0    0    -1
+$EndComp
+Wire Wire Line
+	10550 2350 10550 2450
+NoConn ~ 10050 1350
+Wire Wire Line
+	5500 3150 5700 3150
+Wire Wire Line
+	5500 3250 5700 3250
+Text Label 5700 3150 0    50   ~ 0
+SDA
+Text Label 5700 3250 0    50   ~ 0
+SCL
+$Comp
+L Device:R R7
+U 1 1 5A6CE447
+P 8450 1100
+F 0 "R7" H 8600 1050 50  0000 C CNN
+F 1 "4k7" H 8600 1150 50  0000 C CNN
+F 2 "Resistor_SMD:R_0805_2012Metric" V 8380 1100 50  0001 C CNN
+F 3 "" H 8450 1100 50  0001 C CNN
+	1    8450 1100
+	-1   0    0    1
+$EndComp
+$Comp
+L Device:R R8
+U 1 1 5A6CE6F7
+P 8600 1100
+F 0 "R8" H 8750 1050 50  0000 C CNN
+F 1 "4k7" H 8750 1150 50  0000 C CNN
+F 2 "Resistor_SMD:R_0805_2012Metric" V 8530 1100 50  0001 C CNN
+F 3 "" H 8600 1100 50  0001 C CNN
+	1    8600 1100
+	1    0    0    1
+$EndComp
+Wire Wire Line
+	8450 1250 8450 1350
+Connection ~ 8450 1350
+Wire Wire Line
+	8450 1350 8850 1350
+Wire Wire Line
+	8600 1250 8600 1550
+Wire Wire Line
+	8250 1550 8600 1550
+Connection ~ 8600 1550
+Wire Wire Line
+	8600 1550 8850 1550
+$Comp
+L power:VCC #PWR033
+U 1 1 5A6D9E61
+P 8450 850
+F 0 "#PWR033" H 8450 700 50  0001 C CNN
+F 1 "VCC" H 8467 1023 50  0000 C CNN
+F 2 "" H 8450 850 50  0001 C CNN
+F 3 "" H 8450 850 50  0001 C CNN
+	1    8450 850
+	1    0    0    -1
+$EndComp
+$Comp
+L power:VCC #PWR034
+U 1 1 5A6D9EA6
+P 8600 850
+F 0 "#PWR034" H 8600 700 50  0001 C CNN
+F 1 "VCC" H 8617 1023 50  0000 C CNN
+F 2 "" H 8600 850 50  0001 C CNN
+F 3 "" H 8600 850 50  0001 C CNN
+	1    8600 850
+	1    0    0    -1
+$EndComp
+Wire Wire Line
+	8600 850  8600 950
+Wire Wire Line
+	8450 850  8450 950
 $EndSCHEMATC

Commit message: Start work with pcb
Parts:
- added J6: Output, w_conn_screw:mors_2p, symbol Connector_Generic:Conn_01x02
- J1: value Conn_01x06 -> AVR_ISP
Connections:
- net labels added: AREF, AVCC, RES_ESP
Changed lines of the file:
@@
 P 7150 1300
 F 0 "J1" H 7230 1292 50  0000 L CNN
-F 1 "Conn_01x06" H 7230 1201 50  0000 L CNN
+F 1 "AVR_ISP" H 7230 1201 50  0000 L CNN
 F 2 "Connector_PinHeader_2.54mm:PinHeader_2x03_P2.54mm_Vertical" H 7150 1300 50  0001 C CNN
 F 3 "~" H 7150 1300 50  0001 C CNN
@@
 Wire Wire Line
 	8450 850  8450 950
+Text Label 3200 2200 0    50   ~ 0
+AVCC
+Text Label 7950 2750 0    50   ~ 0
+RES_ESP
+Text Label 3450 2500 2    50   ~ 0
+AREF
+$Comp
+L Connector_Generic:Conn_01x02 J6
+U 1 1 5A7114DD
+P 6250 4800
+F 0 "J6" H 6330 4792 50  0000 L CNN
+F 1 "Output" H 6330 4701 50  0000 L CNN
+F 2 "w_conn_screw:mors_2p" H 6250 4800 50  0001 C CNN
+F 3 "~" H 6250 4800 50  0001 C CNN
+	1    6250 4800
+	1    0    0    -1
+$EndComp
 $EndSCHEMATC

Commit message: Create server witch cfg
Parts:
- added C10, C11: 100n, Capacitor_SMD:C_0805_2012Metric, symbol Device:C
- added J7: Sleep, Connector_PinHeader_2.54mm:PinHeader_1x02_P2.54mm_Vertical, symbol Connector_Generic:Conn_01x02
- added U4: LD1117S33TR_SOT223, Package_TO_SOT_SMD:SOT-223-3_TabPin2, symbol Regulator_Linear:LD1117S33TR_SOT223
Connections:
- net labels added: +5V
- wire segments 127 -> 144
- no-connect marks 23 -> 22
Other:
- moved on the sheet: U1, U3

Commit message: Work with interface
Parts:
- added D1: D, symbol Device:D
- added R9: GL7516, symbol Device:R_PHOTO
- added R?: 27k, symbol Device:R
- added R?: 12k, symbol Device:R
- added R?: 1k, symbol Device:R
Connections:
- net labels added: ADC, ML, MT
- wire segments 144 -> 162
- no-connect marks 22 -> 19
Other:
- note added: "GPIO12(6)"
- note added: "GPIO14(5)"
Changed lines of the file:
@@
 Wire Wire Line
 	8700 3850 8700 4250
-NoConn ~ 7700 4950
-NoConn ~ 7700 5250
-NoConn ~ 7700 5350
 NoConn ~ 7700 5450
 NoConn ~ 10100 5050
@@
 	1    0    0    -1
 $EndComp
+Wire Wire Line
+	7700 4950 7600 4950
+Text Label 7600 4950 0    50   ~ 0
+ADC
+Wire Wire Line
+	3000 6850 3300 6850
+Text Label 3300 6850 0    50   ~ 0
+ADC
+$Comp
+L Device:D D1
+U 1 1 5A94AFAC
+P 3000 7100
+F 0 "D1" V 3046 7021 50  0000 R CNN
+F 1 "D" V 2955 7021 50  0000 R CNN
+F 2 "" H 3000 7100 50  0001 C CNN
+F 3 "~" H 3000 7100 50  0001 C CNN
+	1    3000 7100
+	0    -1   -1   0
+$EndComp
+Wire Wire Line
+	3000 6950 3000 6850
+Wire Wire Line
+	3000 7250 3000 7350
+Wire Wire Line
+	3000 7350 3300 7350
+Wire Wire Line
+	7700 5250 7600 5250
+Text Label 7600 5250 0    50   ~ 0
+MT
+Text Label 3300 7350 0    50   ~ 0
+MT
+$Comp
+L Device:R_PHOTO R9
+U 1 1 5A95D4D8
+P 2400 7100
+F 0 "R9" H 2470 7146 50  0000 L CNN
+F 1 "GL7516" H 2470 7055 50  0000 L CNN
+F 2 "" V 2450 6850 50  0001 L CNN
+F 3 "~" H 2400 7050 50  0001 C CNN
+	1    2400 7100
+	1    0    0    -1
+$EndComp
+Wire Wire Line
+	2400 7250 2400 7450
+Wire Wire Line
+	2400 7450 3300 7450
+Text Label 3300 7450 0    50   ~ 0
+ML
+$Comp
+L Device:R R?
+U 1 1 5A9E4312
+P 2400 6600
+F 0 "R?" H 2330 6554 50  0000 R CNN
+F 1 "27k" H 2330 6645 50  0000 R CNN
+F 2 "" V 2330 6600 50  0001 C CNN
+F 3 "~" H 2400 6600 50  0001 C CNN
+	1    2400 6600
+	-1   0    0    1
+$EndComp
+$Comp
+L Device:R R?
+U 1 1 5A9E441A
+P 2000 7100
+F 0 "R?" H 1930 7054 50  0000 R CNN
+F 1 "12k" H 1930 7145 50  0000 R CNN
+F 2 "" V 1930 7100 50  0001 C CNN
+F 3 "~" H 2000 7100 50  0001 C CNN
+	1    2000 7100
+	-1   0    0    1
+$EndComp
+Wire Wire Line
+	2400 6750 2400 6850
+Wire Wire Line
+	2000 6950 2000 6850
+Wire Wire Line
+	2000 6850 2400 6850
+Connection ~ 2400 6850
+Wire Wire Line
+	2400 6850 2400 6950
+Wire Wire Line
+	2000 7250 2000 7450
+Wire Wire Line
+	2000 7450 2400 7450
+Connection ~ 2400 7450
+$Comp
+L power:VCC #PWR?
+U 1 1 5A9F85FE
+P 2400 6350
+F 0 "#PWR?" H 2400 6200 50  0001 C CNN
+F 1 "VCC" H 2417 6523 50  0000 C CNN
+F 2 "" H 2400 6350 50  0001 C CNN
+F 3 "" H 2400 6350 50  0001 C CNN
+	1    2400 6350
+	1    0    0    -1
+$EndComp
+Wire Wire Line
+	2400 6350 2400 6450
+$Comp
+L Device:R R?
+U 1 1 5AA00198
+P 3000 6600
+F 0 "R?" H 2900 6550 50  0000 C CNN
+F 1 "1k" H 2900 6650 50  0000 C CNN
+F 2 "" V 2930 6600 50  0001 C CNN
+F 3 "~" H 3000 6600 50  0001 C CNN
+	1    3000 6600
+	-1   0    0    1
+$EndComp
+Wire Wire Line
+	7700 5350 7600 5350
+Text Label 7600 5350 0    50   ~ 0
+ML
+Text Notes 3500 7350 0    50   ~ 0
+GPIO14(5)
+Text Notes 3500 7450 0    50   ~ 0
+GPIO12(6)
+Wire Wire Line
+	3000 6750 3000 6850
+Connection ~ 3000 6850
+$Comp
+L power:VCC #PWR?
+U 1 1 5AA1E8BC
+P 3000 6350
+F 0 "#PWR?" H 3000 6200 50  0001 C CNN
+F 1 "VCC" H 3017 6523 50  0000 C CNN
+F 2 "" H 3000 6350 50  0001 C CNN
+F 3 "" H 3000 6350 50  0001 C CNN
+	1    3000 6350
+	1    0    0    -1
+$EndComp
+Wire Wire Line
+	3000 6450 3000 6350
 $EndSCHEMATC

Commit message: Test version
Parts:
- added D?: LED, symbol Device:LED
- added R?: 220, Resistor_SMD:R_0805_2012Metric, symbol Device:R
- D1: footprint (none) -> `
Connections:
- net labels added: LED, MLP, MTP, OUT
- wire segments 162 -> 170
- no-connect marks 19 -> 15
Other:
- note added: "GPIO13(7)"
- note added: "GPIO4(2)"
Changed lines of the file:
@@
 L power:GND #PWR02
 U 1 1 5A6CBB0F
-P 10250 5600
-F 0 "#PWR02" H 10250 5350 50  0001 C CNN
-F 1 "GND" H 10255 5427 50  0000 C CNN
-F 2 "" H 10250 5600 50  0001 C CNN
-F 3 "" H 10250 5600 50  0001 C CNN
-	1    10250 5600
-	1    0    0    -1
-$EndComp
-Wire Wire Line
-	10250 5600 10250 5550
+P 10250 5800
+F 0 "#PWR02" H 10250 5550 50  0001 C CNN
+F 1 "GND" H 10255 5627 50  0000 C CNN
+F 2 "" H 10250 5800 50  0001 C CNN
+F 3 "" H 10250 5800 50  0001 C CNN
+	1    10250 5800
+	1    0    0    -1
+$EndComp
+Wire Wire Line
+	10250 5800 10250 5550
 Wire Wire Line
 	10250 5550 10100 5550
@@
 U 1 1 5A6F0A73
 P 10400 5450
-F 0 "R5" V 10193 5450 50  0000 C CNN
-F 1 "10k" V 10284 5450 50  0000 C CNN
+F 0 "R5" V 10350 5250 50  0000 C CNN
+F 1 "10k" V 10400 5450 50  0000 C CNN
 F 2 "Resistor_SMD:R_0805_2012Metric" V 10330 5450 50  0001 C CNN
 F 3 "" H 10400 5450 50  0001 C CNN
@@
 L power:GND #PWR027
 U 1 1 5A6F5F4B
-P 10600 5600
-F 0 "#PWR027" H 10600 5350 50  0001 C CNN
-F 1 "GND" H 10605 5427 50  0000 C CNN
-F 2 "" H 10600 5600 50  0001 C CNN
-F 3 "" H 10600 5600 50  0001 C CNN
-	1    10600 5600
+P 10600 5800
+F 0 "#PWR027" H 10600 5550 50  0001 C CNN
+F 1 "GND" H 10605 5627 50  0000 C CNN
+F 2 "" H 10600 5800 50  0001 C CNN
+F 3 "" H 10600 5800 50  0001 C CNN
+	1    10600 5800
 	1    0    0    -1
 $EndComp
@@
 	10550 5450 10600 5450
 Wire Wire Line
-	10600 5450 10600 5600
+	10600 5450 10600 5800
 $Comp
 L power:VCC #PWR028
@@
 Wire Wire Line
 	8700 3850 8700 4250
-NoConn ~ 7700 5450
-NoConn ~ 10100 5050
-NoConn ~ 10100 5150
 NoConn ~ 10100 5250
-NoConn ~ 10100 5350
 $Comp
 L maxim:DS1307Z+ U3
@@
 F 0 "D1" V 3046 7021 50  0000 R CNN
 F 1 "D" V 2955 7021 50  0000 R CNN
-F 2 "" H 3000 7100 50  0001 C CNN
+F 2 "`" H 3000 7100 50  0001 C CNN
 F 3 "~" H 3000 7100 50  0001 C CNN
 	1    3000 7100
@@
 	2000 7450 2400 7450
 Connection ~ 2400 7450
-$Comp
-L power:VCC #PWR?
-U 1 1 5A9F85FE
-P 2400 6350
-F 0 "#PWR?" H 2400 6200 50  0001 C CNN
-F 1 "VCC" H 2417 6523 50  0000 C CNN
-F 2 "" H 2400 6350 50  0001 C CNN
-F 3 "" H 2400 6350 50  0001 C CNN
-	1    2400 6350
-	1    0    0    -1
-$EndComp
 Wire Wire Line
 	2400 6350 2400 6450
@@
 	3000 6750 3000 6850
 Connection ~ 3000 6850
-$Comp
-L power:VCC #PWR?
-U 1 1 5AA1E8BC
-P 3000 6350
-F 0 "#PWR?" H 3000 6200 50  0001 C CNN
-F 1 "VCC" H 3017 6523 50  0000 C CNN
-F 2 "" H 3000 6350 50  0001 C CNN
-F 3 "" H 3000 6350 50  0001 C CNN
-	1    3000 6350
-	1    0    0    -1
-$EndComp
 Wire Wire Line
 	3000 6450 3000 6350
+Wire Wire Line
+	2400 6850 3000 6850
+$Comp
+L power:GND #PWR?
+U 1 1 5A9A7E79
+P 10950 5800
+F 0 "#PWR?" H 10950 5550 50  0001 C CNN
+F 1 "GND" H 10955 5627 50  0000 C CNN
+F 2 "" H 10950 5800 50  0001 C CNN
+F 3 "" H 10950 5800 50  0001 C CNN
+	1    10950 5800
+	1    0    0    -1
+$EndComp
+$Comp
+L Device:LED D?
+U 1 1 5A9A7FEE
+P 10950 5550
+F 0 "D?" V 10988 5433 50  0000 R CNN
+F 1 "LED" V 10897 5433 50  0000 R CNN
+F 2 "" H 10950 5550 50  0001 C CNN
+F 3 "~" H 10950 5550 50  0001 C CNN
+	1    10950 5550
+	0    -1   -1   0
+$EndComp
+Wire Wire Line
+	10950 5700 10950 5800
+Wire Wire Line
+	10950 5400 10950 5350
+Text Label 10300 5350 0    50   ~ 0
+LED
+$Comp
+L Device:R R?
+U 1 1 5A9DB11E
+P 10700 5350
+F 0 "R?" V 10650 5550 50  0000 C CNN
+F 1 "220" V 10700 5350 50  0000 C CNN
+F 2 "Resistor_SMD:R_0805_2012Metric" V 10630 5350 50  0001 C CNN
+F 3 "" H 10700 5350 50  0001 C CNN
+	1    10700 5350
+	0    1    1    0
+$EndComp
+Wire Wire Line
+	10100 5350 10550 5350
+Wire Wire Line
+	10850 5350 10950 5350
+Wire Wire Line
+	10100 5050 10300 5050
+Wire Wire Line
+	10100 5150 10300 5150
+Text Label 10300 5050 0    50   ~ 0
+MTP
+Text Label 10300 5150 0    50   ~ 0
+OUT
+Text Label 2400 6350 0    50   ~ 0
+MLP
+Text Label 3000 6350 0    50   ~ 0
+MTP
+Text Notes 2350 6250 0    50   ~ 0
+GPIO13(7)
+Text Notes 2950 6250 0    50   ~ 0
+GPIO4(2)
+Wire Wire Line
+	7700 5450 7600 5450
+Text Label 7600 5450 0    50   ~ 0
+MLP
 $EndSCHEMATC

Commit message: Change schematic for only esp8266
Parts:
- removed BT1: 3V, symbol Device:Battery_Cell
- removed C1, C2: 22p, Capacitor_SMD:C_0603_1608Metric, symbol Device:C
- removed C3, C7, C8: 100n, Capacitor_SMD:C_0805_2012Metric, symbol Device:C
- removed D1: D, `, symbol Device:D
- removed J1: AVR_ISP, Connector_PinHeader_2.54mm:PinHeader_2x03_P2.54mm_Vertical, symbol Connector_Generic:Conn_01x06
- removed J4: AVR_UART, Connector_PinHeader_2.54mm:PinHeader_1x03_P2.54mm_Vertical, symbol Connector_Generic:Conn_01x03
- removed J6: Output, w_conn_screw:mors_2p, symbol Connector_Generic:Conn_01x02
- removed L1: 100u, Inductor_SMD:L_0805_2012Metric, symbol Device:L
- removed R1, R3: 10k, Resistor_SMD:R_0805_2012Metric, symbol Device:R
- removed R2: 1k, Resistor_SMD:R_0805_2012Metric, symbol Device:R
- removed R7, R8: 4k7, Resistor_SMD:R_0805_2012Metric, symbol Device:R
- removed R9: GL7516, symbol Device:R_PHOTO
- removed U1: ATMEGA328-AU, Package_QFP:TQFP-32_7x7mm_P0.8mm, symbol MCU_Atmel_ATMEGA:ATMEGA328-AU
- removed U3: DS1307Z+, Package_SOIC:SO-8_5.3x6.2mm_P1.27mm, symbol maxim:DS1307Z+
- removed Y1: 9,216 MHz, Crystal:Crystal_HC49-4H_Vertical, symbol Device:Crystal
- removed Y2: 32768, Crystal:Crystal_SMD_MicroCrystal_CC4V-T1A-2Pin_5.0x1.9mm, symbol Device:Crystal
- D1: renamed from D?; footprint (none) -> LED_THT:LED_D3.0mm
- R2, R3, R5: renamed from R?; footprint (none) -> Resistor_SMD:R_0805_2012Metric
- gave numbers to parts that had none: 1
- renumbered C5 to C1, C6 to C2, C4 to C3, C10 to C4, C11 to C5, C9 to C6, J7 to J1, J5 to J2, J2 to J3, J3 to J4, R6 to R1, R5 to R7, U4 to U1
Connections:
- net labels removed: AREF, AVCC, LIGHT, MISO, MOSI, RES, SCK, SCL, SDA, TEMP
- wire segments 170 -> 84
- no-connect marks 15 -> 1
Other:
- moved on the sheet: U1

Commit message: Drawing schematic new
Parts:
- removed C2: 100n, Capacitor_SMD:C_0805_2012Metric, symbol Device:C
- removed J3: Temp, w_conn_screw:mors_2p, symbol Connector_Generic:Conn_01x02
- removed R1: 10k, Resistor_SMD:R_0805_2012Metric, symbol Device:R
- added C2: 10u, Capacitor_SMD:CP_Elec_5x5.7, symbol Device:CP
- added C7: 2u2, Capacitor_SMD:C_1812_4532Metric_Pad1.24x3.50mm_HandSolder, symbol Device:C
- added J1: PWR_+5V, Connector_PinHeader_2.54mm:PinHeader_1x02_P2.54mm_Vertical, symbol Connector_Generic:Conn_01x02
- added J5: Sensors, w_conn_screw:mors_3p, symbol Connector_Generic:Conn_01x03
- added Q1: BT139-600, Package_TO_SOT_THT:TO-220-3_Vertical, symbol Triac_Thyristor:BT139-600
- added Q2, Q3: BSS138, Package_TO_SOT_SMD:SOT-23, symbol Transistor_FET:BSS138
- added R10: 330, Resistor_THT:R_Axial_DIN0207_L6.3mm_D2.5mm_P15.24mm_Horizontal, symbol Device:R
- added R11: 470k, Resistor_SMD:R_0805_2012Metric, symbol Device:R
- added R12: 10k, Resistor_SMD:R_0805_2012Metric, symbol Device:R
- added R13: 100k, Resistor_SMD:R_0805_2012Metric, symbol Device:R
- added R5: 240, Resistor_SMD:R_0805_2012Metric, symbol Device:R
- added R8: 51, Resistor_THT:R_Axial_DIN0207_L6.3mm_D2.5mm_P15.24mm_Horizontal, symbol Device:R
- added R9: 10k, Resistor_THT:R_Axial_DIN0207_L6.3mm_D2.5mm_P15.24mm_Horizontal, symbol Device:R
- added SW1: RESET, w_switch:smd_push, symbol Switch:SW_Push
- added U3: MOC3023M, Package_DIP:DIP-6_W7.62mm, symbol Relay_SolidState:MOC3023M
- C5: footprint Capacitor_SMD:C_0805_2012Metric -> Capacitor_THT:C_Axial_L3.8mm_D2.6mm_P7.50mm_Horizontal
- J4: value Light -> OUTPUT
- renumbered J1 to J2, J2 to J3, R2 to R1, R3 to R2, R4 to R3, R5 to R4
Connections:
- net labels added: +3.3V, RESET
- net labels removed: RES_ESP, VCC
- wire segments 84 -> 127
- no-connect marks 1 -> 0
Other:
- moved on the sheet: U1
