File: kicad/grower_light/grower_light.sch (KiCad schematic (older format))
At the start: 33 parts, among them J1 PWR_+5V, J2 Sleep, J3 ESP_UART, J4 OUTPUT, J5 Sensors, Q1 BT139-600, Q2 BSS138, Q3 BSS138, SW1 RESET, U1 LD1117S33TR_SOT223, U2 ESP-12_07v2, U3 MOC3023M

Commit message: Final pcb
Parts:
- removed C4: 100n, Capacitor_SMD:C_0805_2012Metric, symbol Device:C
- removed J4: OUTPUT, w_conn_screw:mors_2p, symbol Connector_Generic:Conn_01x02
- removed J5: Sensors, w_conn_screw:mors_3p, symbol Connector_Generic:Conn_01x03
- added F1: Fuse, Fuse:Fuseholder_TR5_Littlefuse_No560_No460, symbol Device:Fuse
- added J1: AC, Connector_PinHeader_2.54mm:PinHeader_1x02_P2.54mm_Vertical, symbol Connector_Generic:Conn_01x02
- added J4: OUTPUT, w_conn_screw:mors_2p, symbol Connector_Specialized:Screw_Terminal_01x02
- added J7: Sensors, w_conn_screw:mors_3p, symbol Connector_Specialized:Screw_Terminal_01x03
- C3: renamed from C2; footprint Capacitor_SMD:CP_Elec_5x5.7 -> Capacitor_THT:CP_Radial_D5.0mm_P2.50mm
- C6: renamed from C7; footprint Capacitor_SMD:C_1812_4532Metric_Pad1.24x3.50mm_HandSolder -> Capacitor_SMD:C_1206_3216Metric
- J2: value Sleep -> AC_IN; footprint Connector_PinHeader_2.54mm:PinHeader_1x02_P2.54mm_Vertical -> lib:RF-190F
- SW1: footprint w_switch:smd_push -> Button_Switch_THT:SW_Tactile_SPST_Angled_PTS645Vx39-2LFS
- renumbered C3 to C2, C5 to C4, C6 to C5, J1 to J3, J3 to J6, R5 to R1, R7 to R10, R8 to R2, R9 to R3, R10 to R4, R1 to R5, R2 to R6, R3 to R7, R4 to R8, R6 to R9, U3 to U1, U1 to U2, U2 to U3
Connections:
- wire segments 127 -> 130
- no-connect marks 0 -> 1
Other:
- moved on the sheet: C1, C2, C3, C4, J3, Q1, R1, R2, R3, R4, U1, U2

Commit message: Transfer
Parts:
- removed U3: ESP-12_07v2, lib:ESP-07v2, symbol esp-12_07v2_08v2-rescue-esp8266_dht22:ESP-12_07v2_08v2-RESCUE-esp8266_dht22
- added U3: ESP-12_07v2, lib:ESP-07v2, symbol esp-12_07v2_08v2-rescue-esp8266_dht22:ESP-12_07v2
- added U?: DC07-00048A, 7seg:DC07-00048, symbol Lcd7seg:DC07-00048A
Changed lines of the file:
@@
 Text Label 3550 4150 0    50   ~ 0
 MLP
-$Comp
-L esp-12_07v2_08v2-rescue-esp8266_dht22:ESP-12_07v2_08v2-RESCUE-esp8266_dht22 U3
-U 1 1 5A6CB719
-P 4850 3900
-F 0 "U3" H 4850 4643 60  0000 C CNN
-F 1 "ESP-12_07v2" H 4850 4537 60  0000 C CNN
-F 2 "lib:ESP-07v2" H 4850 4431 60  0000 C CNN
-F 3 "" H 4850 3900 60  0000 C CNN
-	1    4850 3900
-	1    0    0    -1
-$EndComp
 Wire Wire Line
 	1900 4700 1450 4700
@@
 	1750 1300 2000 1300
 Connection ~ 2000 1300
+$Comp
+L esp-12_07v2_08v2-rescue-esp8266_dht22:ESP-12_07v2 U3
+U 1 1 5AA73B89
+P 4850 3900
+F 0 "U3" H 4850 4537 60  0000 C CNN
+F 1 "ESP-12_07v2" H 4850 4431 60  0000 C CNN
+F 2 "lib:ESP-07v2" H 4850 3900 60  0000 C CNN
+F 3 "" H 4850 3900 60  0000 C CNN
+	1    4850 3900
+	1    0    0    -1
+$EndComp
+$Comp
+L Lcd7seg:DC07-00048A U?
+U 1 1 5AA89186
+P 9300 3750
+F 0 "U?" H 9225 4315 50  0000 C CNN
+F 1 "DC07-00048A" H 9225 4224 50  0000 C CNN
+F 2 "7seg:DC07-00048" H 9300 3500 50  0001 C CNN
+F 3 "" H 9300 3750 50  0001 C CNN
+	1    9300 3750
+	1    0    0    -1
+$EndComp
 $EndSCHEMATC
