File: kicad/grower_light/grower_light.kicad_pcb (KiCad board)
At the start: 2 copper layers, 20 parts, among them J1 Sleep, J2 ESP_UART, J3 Temp, J4 Light, U1 LD1117S33TR_SOT223, U2 ESP-12_07v2

Commit message: Drawing schematic new
Parts:
- removed C5: 100n, Capacitor_SMD:C_0805_2012Metric
- added J5: Sensors, w_conn_screw:mors_3p, F.Cu at (147.7, 75.7)
- added Q1: BT139-600, Package_TO_SOT_THT:TO-220-3_Vertical, F.Cu at (176.1, 73.1)
- added Q2: BSS138, Package_TO_SOT_SMD:SOT-23, F.Cu at (142.9, 86.4)
- added Q3: BSS138, Package_TO_SOT_SMD:SOT-23, F.Cu at (176.3, 81.3)
- added R11: 470k, Resistor_SMD:R_0805_2012Metric, F.Cu at (166.0, 98.1)
- added R12: 10k, Resistor_SMD:R_0805_2012Metric, F.Cu at (177.5, 87.5)
- added R13: 100k, Resistor_SMD:R_0805_2012Metric, F.Cu at (170.0, 98.6)
- added SW1: RESET, w_switch:smd_push, F.Cu at (167.9, 83.8)
- added U3: MOC3023M, Package_DIP:DIP-6_W7.62mm, F.Cu at (156.8, 71.8)
- C2: value 100n -> 10u; footprint Capacitor_SMD:C_0805_2012Metric -> Capacitor_SMD:CP_Elec_5x5.7
- J1: value Sleep -> PWR_+5V
- J2: value ESP_UART -> Sleep; footprint Connector_PinHeader_2.54mm:PinHeader_1x03_P2.54mm_Vertical -> Connector_PinHeader_2.54mm:PinHeader_1x02_P2.54mm_Vertical
- J3: value Temp -> ESP_UART; footprint w_conn_screw:mors_2p -> Connector_PinHeader_2.54mm:PinHeader_1x03_P2.54mm_Vertical
- J4: value Light -> OUTPUT
- R1: value 10k -> 27k
- R2: value 27k -> 1k
- R3: value 1k -> 100
- R4: value 100 -> 12k
- R5: value 12k -> 240
- moved R7 138.6 mm to (184.8, 80.7)
- moved R6 136.2 mm to (171.4, 93.1)
- moved D1 133.8 mm to (153.9, 95.9)
- moved C1 133.6 mm to (154.7, 102.6)
- moved R4 133.3 mm to (162.2, 98.1)
- moved R2 132.9 mm to (158.6, 102.6)
- moved U1 130.1 mm to (129.1, 95.8)
- moved R1 129.6 mm to (167.8, 90.4)
- moved J2 128.0 mm to (150.4, 95.3)
- moved C4 127.1 mm to (181.4, 86.2)
- moved R3 126.6 mm to (173.9, 87.5)
- moved J1 125.4 mm to (151.9, 86.2)
- moved R5 125.1 mm to (181.1, 80.7)
- moved C3 122.1 mm to (163.9, 92.6)
- moved C6 120.7 mm to (159.8, 92.6)
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Connections:
- C2 pad 1: GND -> +5V
- C2 pad 2: +5V -> GND
- C3 pad 2: VCC -> +3V3
- C4 pad 2: VCC -> +3V3
- C6 pad 1: GND -> /RESET
- C6 pad 2: /RES_ESP -> GND
- J1 pad 1: Net-(J1-Pad1) -> GND
- J1 pad 2: /RES_ESP -> +5V
- J2 pad 1: /TX -> Net-(J2-Pad1)
- J2 pad 2: /RX -> /RESET
- J3 pad 1: /ADC -> /TX
- J3 pad 2: /ML -> /RX
- J4 pad 1: /ADC -> Net-(J4-Pad1)
- J4 pad 2: /MT -> Net-(C5-Pad2)
- R1 pad 1: /RES_ESP -> /ADC
- R1 pad 2: VCC -> /MLP
- R2 pad 2: /MLP -> /MTP
- R3 pad 1: /ADC -> Net-(R3-Pad1)
- R3 pad 2: /MTP -> +3V3
- R4 pad 1: Net-(R4-Pad1) -> /ML
- R4 pad 2: VCC -> /ADC
- R5 pad 1: /ML -> Net-(R5-Pad1)
- R5 pad 2: /ADC -> /OUT
- U1 pad 2: VCC -> +3V3
- U2 pad 1: /RES_ESP -> /RESET
- U2 pad 3: Net-(R4-Pad1) -> Net-(R3-Pad1)
- U2 pad 4: Net-(J1-Pad1) -> Net-(J2-Pad1)
- U2 pad 8: VCC -> +3V3

Commit message: Final pcb
Parts:
- removed J5: Sensors, w_conn_screw:mors_3p
- added C5: 100n, Capacitor_SMD:C_0805_2012Metric, B.Cu at (150.2, 100.3)
- added F1: Fuse, Fuse:Fuseholder_TR5_Littlefuse_No560_No460, F.Cu at (120.7, 83.8)
- added J6: ESP_UART, Connector_PinHeader_2.54mm:PinHeader_1x03_P2.54mm_Vertical, F.Cu at (158.8, 112.4)
- added J7: Sensors, w_conn_screw:mors_3p, F.Cu at (195.6, 110.5)
- added R10: 10k, Resistor_SMD:R_0805_2012Metric, B.Cu at (188.0, 116.5)
- added R8: 12k, Resistor_SMD:R_0805_2012Metric, B.Cu at (191.1, 116.5)
- added R9: 220, Resistor_SMD:R_0805_2012Metric, B.Cu at (188.0, 112.1)
- C1, Q2, Q3, R11, R12, R13: moved to B.Cu
- C2: value 10u -> 100n; footprint Capacitor_SMD:CP_Elec_5x5.7 -> Capacitor_SMD:C_0805_2012Metric; moved to B.Cu
- C3: value 100n -> 10u; footprint Capacitor_SMD:C_0805_2012Metric -> Capacitor_THT:CP_Radial_D5.0mm_P2.50mm
- C4: footprint Capacitor_SMD:C_0805_2012Metric -> Capacitor_THT:C_Axial_L3.8mm_D2.6mm_P7.50mm_Horizontal
- C6: value 100n -> 2u2; footprint Capacitor_SMD:C_0805_2012Metric -> Capacitor_SMD:C_1206_3216Metric; moved to B.Cu
- J1: value PWR_+5V -> AC
- J2: value Sleep -> AC_IN; footprint Connector_PinHeader_2.54mm:PinHeader_1x02_P2.54mm_Vertical -> lib:RF-190F
- J3: value ESP_UART -> PWR_+5V; footprint Connector_PinHeader_2.54mm:PinHeader_1x03_P2.54mm_Vertical -> Connector_PinHeader_2.54mm:PinHeader_1x02_P2.54mm_Vertical
- R1: value 27k -> 240; moved to B.Cu
- R2: value 1k -> 51; footprint Resistor_SMD:R_0805_2012Metric -> Resistor_THT:R_Axial_DIN0207_L6.3mm_D2.5mm_P15.24mm_Horizontal
- R3: value 100 -> 10k; footprint Resistor_SMD:R_0805_2012Metric -> Resistor_THT:R_Axial_DIN0207_L6.3mm_D2.5mm_P15.24mm_Horizontal
- R4: value 12k -> 330; footprint Resistor_SMD:R_0805_2012Metric -> Resistor_THT:R_Axial_DIN0207_L6.3mm_D2.5mm_P15.24mm_Horizontal
- R5: value 240 -> 27k; moved to B.Cu
- R6: value 220 -> 1k; moved to B.Cu
- R7: value 10k -> 100; moved to B.Cu
- SW1: footprint w_switch:smd_push -> Button_Switch_THT:SW_Tactile_SPST_Angled_PTS645Vx39-2LFS
- U1: value LD1117S33TR_SOT223 -> MOC3023M; footprint Package_TO_SOT_SMD:SOT-223-3_TabPin2 -> Package_DIP:DIP-6_W7.62mm
- U2: value ESP-12_07v2 -> LD1117S33TR_SOT223; footprint lib:ESP-07v2 -> Package_TO_SOT_SMD:SOT-223-3_TabPin2; moved to B.Cu
- U3: value MOC3023M -> ESP-12_07v2; footprint Package_DIP:DIP-6_W7.62mm -> lib:ESP-07v2; moved to B.Cu
- moved C4 74.3 mm to (111.6, 111.8), turned to 180 degrees
- moved Q1 53.3 mm to (127.6, 95.2), turned to 270 degrees
- moved R3 48.5 mm to (130.8, 109.9), turned to 180 degrees
- moved J2 47.3 mm to (103.3, 91.0), turned to 90 degrees
- moved R4 43.6 mm to (119.4, 106.0), turned to 180 degrees
- moved R2 41.5 mm to (119.4, 116.2), turned to 180 degrees
- moved U3 40.9 mm to (174.6, 108.6), turned to 270 degrees
- moved SW1 36.8 mm to (153.0, 117.5), turned to 180 degrees
- moved D1 36.7 mm to (190.5, 98.4), turned to 270 degrees
- moved R1 36.3 mm to (143.5, 117.5)
- moved Q3 35.7 mm to (150.2, 105.7)
- moved R7 33.1 mm to (159.5, 102.0), turned to 270 degrees
- moved J3 32.9 mm to (143.5, 92.1), turned to 270 degrees
- moved C3 30.7 mm to (141.0, 113.0)
- moved C2 30.1 mm to (186.1, 99.4), turned to 270 degrees
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Connections:
- C2 pad 1: +5V -> GND
- C2 pad 2: GND -> +3V3
- C3 pad 1: GND -> +3V3
- C3 pad 2: +3V3 -> GND
- C4 pad 1: GND -> Net-(C4-Pad1)
- C4 pad 2: +3V3 -> Net-(C4-Pad2)
- C6 pad 1: /RESET -> Net-(C6-Pad1)
- J1 pad 1: GND -> Net-(C4-Pad2)
- J1 pad 2: +5V -> Net-(F1-Pad1)
- J2 pad 1: Net-(J2-Pad1) -> Net-(C4-Pad2)
- J2 pad 2: /RESET -> Net-(F1-Pad2)
- J3 pad 1: /TX -> GND
- J3 pad 2: /RX -> +5V
- J4 pad 1: Net-(J4-Pad1) -> Net-(F1-Pad1)
- J4 pad 2: Net-(C5-Pad2) -> Net-(J4-Pad2)
- Q1 pad 1: Net-(C5-Pad2) -> Net-(C4-Pad2)
- Q1 pad 2: Net-(J4-Pad1) -> Net-(J4-Pad2)
- Q3 pad 1: Net-(C7-Pad1) -> Net-(C6-Pad1)
- R1 pad 1: /ADC -> Net-(R1-Pad1)
- R1 pad 2: /MLP -> /OUT
- R13 pad 1: Net-(C7-Pad1) -> Net-(C6-Pad1)
- R2 pad 1: /ADC -> Net-(J4-Pad2)
- R2 pad 2: /MTP -> Net-(C4-Pad1)
- R3 pad 2: +3V3 -> Net-(Q1-Pad3)
- R4 pad 1: /ML -> Net-(Q1-Pad3)
- R4 pad 2: /ADC -> Net-(C4-Pad2)
- R5 pad 1: Net-(R5-Pad1) -> /ADC
- R5 pad 2: /OUT -> /MLP
- R6 pad 1: Net-(D1-Pad2) -> /ADC
- R6 pad 2: /LED -> /MTP
- R7 pad 1: GND -> Net-(R7-Pad1)
- R7 pad 2: Net-(R7-Pad2) -> +3V3
- SW1 pad 1: GND -> /RESET
- SW1 pad 2: /RESET -> GND
- U1 pad 1: GND -> Net-(R1-Pad1)
- U1 pad 2: +3V3 -> GND
- U1 pad 3: +5V -> Net-(U1-Pad3)
- U2 pad 1: /RESET -> GND
- U2 pad 2: /ADC -> +3V3
- U2 pad 3: Net-(R3-Pad1) -> +5V
- U3 pad 1: Net-(R5-Pad1) -> /RESET
- U3 pad 2: GND -> /ADC
- U3 pad 3: Net-(U3-Pad3) -> Net-(R7-Pad1)
- U3 pad 5: Net-(U3-Pad5) -> /MT
- U3 pad 6: Net-(J4-Pad1) -> /ML
Routing:
- net GND: track 0.00 -> 148.3 mm
- net +3V3: track 0.00 -> 76.0 mm, vias 0 -> 4
- net /RESET: track 0.00 -> 54.7 mm
- net Net-(F1-Pad1): track 0.00 -> 49.7 mm
- net Net-(C4-Pad2): track 0.00 -> 47.6 mm
- net /ADC: track 0.00 -> 43.3 mm
- net Net-(J4-Pad2): track 0.00 -> 41.3 mm
- net /OUT: track 0.00 -> 39.9 mm
- net Net-(Q3-Pad3): track 0.00 -> 38.6 mm
- net /ML: track 0.00 -> 37.5 mm, vias 0 -> 2
- net Net-(R1-Pad1): track 0.00 -> 31.7 mm
- net Net-(R3-Pad1): track 0.00 -> 28.4 mm
- net /MT: track 0.00 -> 26.9 mm
- net +5V: track 0.00 -> 19.2 mm
- net Net-(R7-Pad1): track 0.00 -> 16.2 mm
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Other:
- board outline added: 98 x 41 mm
- board text added: "BOT"
